Commit message: v1.3 workspace sync: API cleanup, localization/planning integration updates

File: camrod_sensor_kit/urdf/camrod_sensor_kit.xacro (robot description, xacro)
@@ -1,11 +1,20 @@
 <?xml version="1.0"?>
-<!-- HH_251215: camping cart sensor kit URDF -->
 <robot name="camrod_sensor_kit" xmlns:xacro="http://www.ros.org/wiki/xacro">
+  <!-- ========================================================= -->
+  <!-- 1. Base link / sensor kit base link arguments             -->
+  <!-- ========================================================= -->
   <xacro:arg name="base_link" default="robot_base_link"/>
-  <!-- HH_260220: Introduce a dedicated sensor kit anchor frame under robot_base_link. -->
   <xacro:arg name="sensor_kit_base_link" default="sensor_kit_base_link"/>
+  <!-- ========================================================= -->
+  <!-- 2. Simple robot body size (for visualization only)        -->
+  <!-- ========================================================= -->
   <xacro:arg name="base_length" default="1.4"/>
-  <xacro:arg name="base_width" default="0.7"/>
+  <xacro:arg name="base_width"  default="0.7"/>
   <xacro:arg name="base_height" default="1.2"/>
+  <!-- ========================================================= -->
+  <!-- 3. Existing sensor transform arguments                    -->
+  <!--    xyz: meters                                            -->
+  <!--    rpy: radians                                           -->
+  <!-- ========================================================= -->
   <xacro:arg name="imu_xyz" default="0.1 0.0 0.4"/>
   <xacro:arg name="imu_rpy" default="0.0 0.0 0.0"/>
@@ -14,17 +23,50 @@
   <xacro:arg name="lidar_xyz" default="0.5 0.0 0.5"/>
   <xacro:arg name="lidar_rpy" default="0.0 0.0 0.0"/>
-  <xacro:arg name="camera_front_xyz" default="0.45 0.0 0.8"/>
-  <xacro:arg name="camera_front_rpy" default="-0.087266 0.0 0.0"/>
+  <!-- HH_260326: Canonical camera frame arguments. -->
+  <xacro:arg name="camera_xyz" default="0.35 0.0 0.8"/>
+  <xacro:arg name="camera_rpy" default="0.0 0.0 0.0"/>
+  <!-- HH_260326: Optional aggregate radar frame under sensor_kit_base_link. -->
+  <xacro:arg name="radar_xyz" default="0.0 0.0 0.0"/>
+  <xacro:arg name="radar_rpy" default="0.0 0.0 0.0"/>
+  <!-- ========================================================= -->
+  <!-- 4. Radar transform arguments                              -->
+  <!--    yaw examples:                                          -->
+  <!--      front  =   0 deg =  0.0                              -->
+  <!--      left1  =  90 deg =  1.570796                         -->
+  <!--      left2  = 135 deg =  2.356194                         -->
+  <!--      right1 = -90 deg = -1.570796                         -->
+  <!--      right2 = -135deg = -2.356194                         -->
+  <!--      rear   = 180 deg =  3.141593                         -->
+  <!-- ========================================================= -->
+  <xacro:arg name="radar_front_xyz"  default="0.55 0.0 0.45"/>
+  <xacro:arg name="radar_front_rpy"  default="0.0 0.0 0.0"/>
+  <xacro:arg name="radar_left1_xyz"  default="0.20 0.45 0.45"/>
+  <xacro:arg name="radar_left1_rpy"  default="0.0 0.0 1.570796"/>
+  <xacro:arg name="radar_left2_xyz"  default="-0.20 0.45 0.45"/>
+  <xacro:arg name="radar_left2_rpy"  default="0.0 0.0 2.356194"/>
+  <xacro:arg name="radar_right1_xyz" default="0.20 -0.45 0.45"/>
+  <xacro:arg name="radar_right1_rpy" default="0.0 0.0 -1.570796"/>
+  <xacro:arg name="radar_right2_xyz" default="-0.20 -0.45 0.45"/>
+  <xacro:arg name="radar_right2_rpy" default="0.0 0.0 -2.356194"/>
+  <xacro:arg name="radar_rear_xyz"   default="-0.55 0.0 0.45"/>
+  <xacro:arg name="radar_rear_rpy"   default="0.0 0.0 3.141593"/>
+  <!-- ========================================================= -->
+  <!-- 5. Local properties                                       -->
+  <!-- ========================================================= -->
   <xacro:property name="base_link_name" value="$(arg base_link)"/>
   <xacro:property name="sensor_kit_base_link_name" value="$(arg sensor_kit_base_link)"/>
   <xacro:property name="base_length_val" value="$(arg base_length)"/>
-  <xacro:property name="base_width_val" value="$(arg base_width)"/>
+  <xacro:property name="base_width_val"  value="$(arg base_width)"/>
   <xacro:property name="base_height_val" value="$(arg base_height)"/>
-  <xacro:macro name="sensor_link" params="name parent xyz rpy color_rgba">
+  <!-- ========================================================= -->
+  <!-- 6. Reusable sensor macro                                  -->
+  <!--    Creates one link + one fixed joint                     -->
+  <!-- ========================================================= -->
+  <xacro:macro name="sensor_link" params="name parent xyz rpy color_rgba radius length mass">
     <link name="${name}">
       <visual>
         <origin xyz="0 0 0" rpy="0 0 0"/>
         <geometry>
-          <cylinder radius="0.04" length="0.08"/>
+          <cylinder radius="${radius}" length="${length}"/>
         </geometry>
         <material name="${name}_mat">
@@ -35,11 +77,13 @@
         <origin xyz="0 0 0" rpy="0 0 0"/>
         <geometry>
-          <cylinder radius="0.04" length="0.08"/>
+          <cylinder radius="${radius}" length="${length}"/>
         </geometry>
       </collision>
       <inertial>
-        <mass value="0.1"/>
+        <mass value="${mass}"/>
         <origin xyz="0 0 0" rpy="0 0 0"/>
-        <inertia ixx="1e-4" ixy="0" ixz="0" iyy="1e-4" iyz="0" izz="1e-4"/>
+        <inertia ixx="1e-4" ixy="0.0" ixz="0.0"
+                 iyy="1e-4" iyz="0.0"
+                 izz="1e-4"/>
       </inertial>
     </link>
@@ -50,23 +94,34 @@
     </joint>
   </xacro:macro>
+  <!-- ========================================================= -->
+  <!-- 7. Robot base link                                        -->
+  <!-- ========================================================= -->
   <link name="${base_link_name}">
     <visual>
-      <origin xyz="0 0 ${base_height_val/2}" rpy="0 0 0"/>
+      <origin xyz="0 0 ${base_height_val / 2.0}" rpy="0 0 0"/>
       <geometry>
         <box size="${base_length_val} ${base_width_val} ${base_height_val}"/>
       </geometry>
       <material name="body_color">
-        <color rgba="0.1 0.6 0.9 0.2"/>
+        <color rgba="0.10 0.60 0.90 0.20"/>
       </material>
     </visual>
     <collision>
-      <origin xyz="0 0 ${base_height_val/2}" rpy="0 0 0"/>
+      <origin xyz="0 0 ${base_height_val / 2.0}" rpy="0 0 0"/>
       <geometry>
         <box size="${base_length_val} ${base_width_val} ${base_height_val}"/>
       </geometry>
     </collision>
-    <!-- KDL parser in ROS2 warns when the root link has inertia.
-         This URDF is used for TF/visualization, so root-link inertial is omitted. -->
+    <inertial>
+      <mass value="10.0"/>
+      <origin xyz="0 0 ${base_height_val / 2.0}" rpy="0 0 0"/>
+      <inertia ixx="1.0" ixy="0.0" ixz="0.0"
+               iyy="1.0" iyz="0.0"
+               izz="1.0"/>
+    </inertial>
   </link>
+  <!-- ========================================================= -->
+  <!-- 8. Sensor kit base link                                   -->
+  <!-- ========================================================= -->
   <link name="${sensor_kit_base_link_name}"/>
   <joint name="${base_link_name}_to_${sensor_kit_base_link_name}" type="fixed">
@@ -75,8 +130,106 @@
     <origin xyz="0 0 0" rpy="0 0 0"/>
   </joint>
-  <!-- HH_260220: Keep only the active sensing stack frames on the sensor kit tree. -->
-  <xacro:sensor_link name="imu_link" parent="${sensor_kit_base_link_name}" xyz="$(arg imu_xyz)" rpy="$(arg imu_rpy)" color_rgba="1.0 0.8 0.2 1.0"/>
-  <xacro:sensor_link name="gnss_link" parent="${sensor_kit_base_link_name}" xyz="$(arg gnss_xyz)" rpy="$(arg gnss_rpy)" color_rgba="0.6 0.9 0.4 1.0"/>
-  <xacro:sensor_link name="lidar_link" parent="${sensor_kit_base_link_name}" xyz="$(arg lidar_xyz)" rpy="$(arg lidar_rpy)" color_rgba="0.9 0.3 0.3 1.0"/>
-  <xacro:sensor_link name="camera_front_link" parent="${sensor_kit_base_link_name}" xyz="$(arg camera_front_xyz)" rpy="$(arg camera_front_rpy)" color_rgba="0.3 0.7 0.95 1.0"/>
+  <!-- ========================================================= -->
+  <!-- 9. Existing sensors                                       -->
+  <!-- ========================================================= -->
+  <xacro:sensor_link
+    name="imu_link"
+    parent="${sensor_kit_base_link_name}"
+    xyz="$(arg imu_xyz)"
+    rpy="$(arg imu_rpy)"
+    color_rgba="1.0 0.8 0.2 1.0"
+    radius="0.03"
+    length="0.06"
+    mass="0.10"/>
+  <xacro:sensor_link
+    name="gnss_link"
+    parent="${sensor_kit_base_link_name}"
+    xyz="$(arg gnss_xyz)"
+    rpy="$(arg gnss_rpy)"
+    color_rgba="0.6 0.9 0.4 1.0"
+    radius="0.03"
+    length="0.06"
+    mass="0.10"/>
+  <xacro:sensor_link
+    name="lidar_link"
+    parent="${sensor_kit_base_link_name}"
+    xyz="$(arg lidar_xyz)"
+    rpy="$(arg lidar_rpy)"
+    color_rgba="0.9 0.3 0.3 1.0"
+    radius="0.05"
+    length="0.10"
+    mass="0.30"/>
+  <xacro:sensor_link
+    name="camera_link"
+    parent="${sensor_kit_base_link_name}"
+    xyz="$(arg camera_xyz)"
+    rpy="$(arg camera_rpy)"
+    color_rgba="0.4 0.8 1.0 1.0"
+    radius="0.04"
+    length="0.08"
+    mass="0.15"/>
+  <!-- ========================================================= -->
+  <!-- 10. Radar sensors                                         -->
+  <!-- ========================================================= -->
+  <!-- HH_260326: Group radar sensors under radar_link frame. -->
+  <link name="radar_link"/>
+  <joint name="radar_link_joint" type="fixed">
+    <parent link="${sensor_kit_base_link_name}"/>
+    <child link="radar_link"/>
+    <origin xyz="$(arg radar_xyz)" rpy="$(arg radar_rpy)"/>
+  </joint>
+  <xacro:sensor_link
+    name="radar_front_link"
+    parent="radar_link"
+    xyz="$(arg radar_front_xyz)"
+    rpy="$(arg radar_front_rpy)"
+    color_rgba="0.95 0.65 0.20 1.0"
+    radius="0.03"
+    length="0.06"
+    mass="0.10"/>
+  <xacro:sensor_link
+    name="radar_left1_link"
+    parent="radar_link"
+    xyz="$(arg radar_left1_xyz)"
+    rpy="$(arg radar_left1_rpy)"
+    color_rgba="0.95 0.65 0.20 1.0"
+    radius="0.03"
+    length="0.06"
+    mass="0.10"/>
+  <xacro:sensor_link
+    name="radar_left2_link"
+    parent="radar_link"
+    xyz="$(arg radar_left2_xyz)"
+    rpy="$(arg radar_left2_rpy)"
+    color_rgba="0.95 0.65 0.20 1.0"
+    radius="0.03"
+    length="0.06"
+    mass="0.10"/>
+  <xacro:sensor_link
+    name="radar_right1_link"
+    parent="radar_link"
+    xyz="$(arg radar_right1_xyz)"
+    rpy="$(arg radar_right1_rpy)"
+    color_rgba="0.95 0.65 0.20 1.0"
+    radius="0.03"
+    length="0.06"
+    mass="0.10"/>
+  <xacro:sensor_link
+    name="radar_right2_link"
+    parent="radar_link"
+    xyz="$(arg radar_right2_xyz)"
+    rpy="$(arg radar_right2_rpy)"
+    color_rgba="0.95 0.65 0.20 1.0"
+    radius="0.03"
+    length="0.06"
+    mass="0.10"/>
+  <xacro:sensor_link
+    name="radar_rear_link"
+    parent="radar_link"
+    xyz="$(arg radar_rear_xyz)"
+    rpy="$(arg radar_rear_rpy)"
+    color_rgba="0.95 0.65 0.20 1.0"
+    radius="0.03"
+    length="0.06"
+    mass="0.10"/>
 </robot>

Commit message: Release v1.6: update CAMROD workspace contents

File: camrod_sensor_kit/urdf/camrod_sensor_kit.xacro (robot description, xacro)
@@ -4,5 +4,5 @@
   <!-- 1. Base link / sensor kit base link arguments             -->
   <!-- ========================================================= -->
-  <xacro:arg name="base_link" default="robot_base_link"/>
+  <xacro:arg name="robot_base_link" default="robot_base_link"/>
   <xacro:arg name="sensor_kit_base_link" default="sensor_kit_base_link"/>
   <!-- ========================================================= -->
@@ -54,5 +54,5 @@
   <!-- 5. Local properties                                       -->
   <!-- ========================================================= -->
-  <xacro:property name="base_link_name" value="$(arg base_link)"/>
+  <xacro:property name="base_link_name" value="$(arg robot_base_link)"/>
   <xacro:property name="sensor_kit_base_link_name" value="$(arg sensor_kit_base_link)"/>
   <xacro:property name="base_length_val" value="$(arg base_length)"/>

Commit message: Release v1.8: ESKF stability, GNSS COG auto-init, DR timeout, platform fixes
localization:
- Replace all Kalman updates with Joseph form to guarantee positive semi-definite covariance
- Add gnss_cog_force_init: hard-reset yaw from first valid COG, eliminating manual offset calibration
- Fix is_stopped_ default (true→false) — permanent yaw freeze when wheel odom absent
- Lower gnss_cog_min_speed_mps 1.5→0.8 to match platform max speed (~1.1 m/s)
- Add publish_uninitialized_tf to keep TF tree connected before GNSS init
- Add DR timeout and covariance-trace gate in localization_monitor_node

planning:
- Add speed_scale parameter to cmd_vel_gate (default 0.5 for safety)
- Implement navigate_to_pose with planner selector for grid/lanelet switching
- Add DR timeout integration in cmd_vel_gate_node

platform:
- robot_visualization_node: publish marker arrays for operator display
- ranger_platform_bridge_node: minor status fixes

util:
- Add gnss_imu_direction_check.py diagnostic script (NavPVT + IMU yaw comparison)

config/map:
- Update lanelet2_maps.osm with latest field survey data
- Update camping_sites, drop_zones, map_info for current deployment site

File: camrod_sensor_kit/urdf/camrod_sensor_kit.xacro (robot description, xacro)
@@ -26,7 +26,4 @@
   <xacro:arg name="camera_xyz" default="0.35 0.0 0.8"/>
   <xacro:arg name="camera_rpy" default="0.0 0.0 0.0"/>
-  <!-- HH_260326: Optional aggregate radar frame under sensor_kit_base_link. -->
-  <xacro:arg name="radar_xyz" default="0.0 0.0 0.0"/>
-  <xacro:arg name="radar_rpy" default="0.0 0.0 0.0"/>
   <!-- ========================================================= -->
   <!-- 4. Radar transform arguments                              -->
@@ -172,14 +169,8 @@
   <!-- 10. Radar sensors                                         -->
   <!-- ========================================================= -->
-  <!-- HH_260326: Group radar sensors under radar_link frame. -->
-  <link name="radar_link"/>
-  <joint name="radar_link_joint" type="fixed">
-    <parent link="${sensor_kit_base_link_name}"/>
-    <child link="radar_link"/>
-    <origin xyz="$(arg radar_xyz)" rpy="$(arg radar_rpy)"/>
-  </joint>
+  <!-- HH_260507: Radar sensors are attached directly under sensor_kit_base_link. -->
   <xacro:sensor_link
     name="radar_front_link"
-    parent="radar_link"
+    parent="${sensor_kit_base_link_name}"
     xyz="$(arg radar_front_xyz)"
     rpy="$(arg radar_front_rpy)"
@@ -190,5 +181,5 @@
   <xacro:sensor_link
     name="radar_left1_link"
-    parent="radar_link"
+    parent="${sensor_kit_base_link_name}"
     xyz="$(arg radar_left1_xyz)"
     rpy="$(arg radar_left1_rpy)"
@@ -199,5 +190,5 @@
   <xacro:sensor_link
     name="radar_left2_link"
-    parent="radar_link"
+    parent="${sensor_kit_base_link_name}"
     xyz="$(arg radar_left2_xyz)"
     rpy="$(arg radar_left2_rpy)"
@@ -208,5 +199,5 @@
   <xacro:sensor_link
     name="radar_right1_link"
-    parent="radar_link"
+    parent="${sensor_kit_base_link_name}"
     xyz="$(arg radar_right1_xyz)"
     rpy="$(arg radar_right1_rpy)"
@@ -217,5 +208,5 @@
   <xacro:sensor_link
     name="radar_right2_link"
-    parent="radar_link"
+    parent="${sensor_kit_base_link_name}"
     xyz="$(arg radar_right2_xyz)"
     rpy="$(arg radar_right2_rpy)"
@@ -226,5 +217,5 @@
   <xacro:sensor_link
     name="radar_rear_link"
-    parent="radar_link"
+    parent="${sensor_kit_base_link_name}"
     xyz="$(arg radar_rear_xyz)"
     rpy="$(arg radar_rear_rpy)"

Commit message: refactor(HH_260528): dual econ camera, unified IMU, platform/planning cleanup
[camrod_sensing]
- camera.launch.py: 전방/후방 카메라 분리 — camera_front_publisher_node (GPU VPI+NvJPEG),
  camera_rear_publisher_node (CPU OpenCV+GStreamer); __yaml__ sentinel으로 camera_params.yaml에서
  enable_front/rear_camera 읽어 OpaqueFunction으로 활성화 결정
- camera_front_publisher_node.cpp/.hpp: camera_publisher_node에서 rename,
  클래스명 CameraFrontPublisherNode, PLUGIN 등록명 일치 수정
- camera_rear_publisher_node.cpp: 신규 추가 — image_raw + image_raw/compressed 발행,
  Isaac ROS AprilTag 도킹용 미압축 스트림 지원
- CMakeLists.txt: camera_publisher_component → camera_front_publisher_component,
  rear 노드 빌드 추가 (cv_bridge, yaml-cpp)
- imu.launch.py: imu_cv7 / imu_gq7_ntrip 두 파일 통합 → imu_model 파라미터로
  cv7(직접 노드, respawn) / gq7(microstrain_launch.py + NTRIP) 분기
- sensing.launch.py: imu_mode → imu_model, cv7/gq7_param_file → imu_param_file,
  enable_front/rear_camera 인자 추가
- config/camera/camera_params.yaml: 전방/후방 FQN별 파라미터 분리,
  camrod_sensing_camera 섹션(활성화 플래그) 추가
- 레거시 삭제: imu_cv7.launch.py, imu_gq7_ntrip.launch.py, camera_publisher_node.cpp/.hpp,
  *_copy_org/750/722 백업 파일 6개

[camrod_bringup]
- launch_defaults.yaml: sensing 섹션 — imu_model/imu_param_file 추가, cv7/gq7_param_file 제거,
  enable_front/rear_camera 추가, camera_params_file 경로 수정
- _bringup_impl.py: OVERRIDE_SPECS sensing에 imu_param_file/camera_params_file 추가,
  arg_specs에 imu_model/enable_front/rear_camera 추가; 비파일 값(bool, 모델명)은
  OVERRIDE_SPECS에서 제거하여 bogus path resolve 방지
- config/sensing/camera/camera_params.yaml: 신규 — bringup 수준 배포별 카메라 override
- config/system/diagnostics/default/sensing/camera_checker.yaml: 전방 image_rect/compressed,
  후방 image_raw/compressed 토픽으로 갱신
- config/sensor_kit/robot_params.yaml: 전/후방 카메라 TF 위치 갱신
- config/planning/nav2_base.yaml: costmap_wait_timeout 12s→2.5s, Smac 계획 시간 상한 추가
- config/planning/goal_replanner.yaml: 파라미터 정리
- 레거시 삭제: nav2_vehicle(copy_org).yaml, sensing/*_copy 파일 3개

[camrod_sensor_kit]
- camrod_sensor_kit.xacro: econ_camera_link 매크로 추가 (body + optical 프레임 쌍 생성),
  전/후방 카메라 arg 및 link/joint 추가 (camera_front_link, camera_rear_link)
- robot_params.yaml: camera_front/rear_xyz/rpy 값 추가
- sensor_kit.launch.py: xacro에 camera_front/rear 인자 전달

[camrod_docking]
- docking.launch.py: 중복 static_transform_publisher 4개 제거 — camera TF는 이제
  sensor_kit(robot_state_publisher)에서 발행하므로 docking에서 중복 불필요

[camrod_platform]
- platform.launch.py: platform_type, ranger_bridge_enable, sensor_kit_bridge_enable 인자 추가
- ranger.launch.py: enable_ranger_base_node / enable_ranger_bridge_node 분리 토글 지원

[camrod_planning]
- nav2_base.yaml: costmap_wait_timeout 12s→2.5s, Smac2D max_planning_time 상한 추가
- goal_replanner.launch.py: launch 내 하드코딩 파라미터 제거, yaml 파일로 제어
- nav2_combo_profiles/*.yaml: 프로파일 정리

[camrod_system]
- config/diagnostics/default/sensing/camera_checker.yaml: 전/후방 카메라 토픽 갱신

File: camrod_sensor_kit/urdf/camrod_sensor_kit.xacro (robot description, xacro)
@@ -26,4 +26,13 @@
   <xacro:arg name="camera_xyz" default="0.35 0.0 0.8"/>
   <xacro:arg name="camera_rpy" default="0.0 0.0 0.0"/>
+  <!-- HH_260528: Dual econ camera arguments (front + rear).                    -->
+  <!--   TF: sensor_kit_base_link → camera_front_link → camera_front (optical) -->
+  <!--       sensor_kit_base_link → camera_rear_link  → camera_rear  (optical) -->
+  <!--   front: x=0.40 m, z=0.46 m, yaw=0 (forward-facing)                    -->
+  <!--   rear : x=0.10 m, z=0.46 m, yaw=π (backward-facing)                   -->
+  <xacro:arg name="camera_front_xyz" default="0.40 0.0 0.46"/>
+  <xacro:arg name="camera_front_rpy" default="0.0 0.0 0.0"/>
+  <xacro:arg name="camera_rear_xyz"  default="0.10 0.0 0.46"/>
+  <xacro:arg name="camera_rear_rpy"  default="0.0 0.0 3.141593"/>
   <!-- ========================================================= -->
   <!-- 4. Radar transform arguments                              -->
@@ -57,7 +66,7 @@
   <xacro:property name="base_height_val" value="$(arg base_height)"/>
   <!-- ========================================================= -->
-  <!-- 6. Reusable sensor macro                                  -->
-  <!--    Creates one link + one fixed joint                     -->
-  <!-- ========================================================= -->
+  <!-- 6. Reusable sensor macros                                 -->
+  <!-- ========================================================= -->
+  <!-- sensor_link: one body link + one fixed joint -->
   <xacro:macro name="sensor_link" params="name parent xyz rpy color_rgba radius length mass">
     <link name="${name}">
@@ -89,4 +98,46 @@
       <child link="${name}"/>
       <origin xyz="${xyz}" rpy="${rpy}"/>
+    </joint>
+  </xacro:macro>
+  <!-- HH_260528: econ_camera_link macro                                       -->
+  <!--   Creates a body frame (name) and an optical child frame (optical_name).-->
+  <!--   optical_name joint uses the standard ROS camera optical convention:  -->
+  <!--     RPY = -π/2, 0, -π/2  (Z forward, Y down in optical frame)         -->
+  <xacro:macro name="econ_camera_link" params="name optical_name parent xyz rpy">
+    <link name="${name}">
+      <visual>
+        <origin xyz="0 0 0" rpy="0 0 0"/>
+        <geometry>
+          <box size="0.06 0.10 0.04"/>
+        </geometry>
+        <material name="${name}_mat">
+          <color rgba="0.15 0.15 0.15 1.0"/>
+        </material>
+      </visual>
+      <collision>
+        <origin xyz="0 0 0" rpy="0 0 0"/>
+        <geometry>
+          <box size="0.06 0.10 0.04"/>
+        </geometry>
+      </collision>
+      <inertial>
+        <mass value="0.15"/>
+        <origin xyz="0 0 0" rpy="0 0 0"/>
+        <inertia ixx="1e-4" ixy="0.0" ixz="0.0"
+                 iyy="1e-4" iyz="0.0"
+                 izz="1e-4"/>
+      </inertial>
+    </link>
+    <joint name="${name}_joint" type="fixed">
+      <parent link="${parent}"/>
+      <child link="${name}"/>
+      <origin xyz="${xyz}" rpy="${rpy}"/>
+    </joint>
+    <!-- Optical frame: Z forward, Y down (standard ROS camera convention). -->
+    <link name="${optical_name}"/>
+    <joint name="${optical_name}_joint" type="fixed">
+      <parent link="${name}"/>
+      <child link="${optical_name}"/>
+      <origin xyz="0 0 0" rpy="-1.570796 0.0 -1.570796"/>
     </joint>
   </xacro:macro>
@@ -224,3 +275,20 @@
     length="0.06"
     mass="0.10"/>
+  <!-- ========================================================= -->
+  <!-- 11. Econ dual cameras (HH_260528)                         -->
+  <!--     sensor_kit_base_link → camera_front_link → camera_front -->
+  <!--     sensor_kit_base_link → camera_rear_link  → camera_rear  -->
+  <!-- ========================================================= -->
+  <xacro:econ_camera_link
+    name="camera_front_link"
+    optical_name="camera_front"
+    parent="${sensor_kit_base_link_name}"
+    xyz="$(arg camera_front_xyz)"
+    rpy="$(arg camera_front_rpy)"/>
+  <xacro:econ_camera_link
+    name="camera_rear_link"
+    optical_name="camera_rear"
+    parent="${sensor_kit_base_link_name}"
+    xyz="$(arg camera_rear_xyz)"
+    rpy="$(arg camera_rear_rpy)"/>
 </robot>
